File: kicad/FreeFi232Large/FreeFi232Large.kicad_pcb (KiCad board)
At the start: 2 copper layers, 40.6 x 53.3 mm, 58 parts, among them J1 DB25-Female, J2 3V3-SERIAL, J3 HWFLOW, J4 USB_OTG, J5 ALT-POWER, SW1 B3S-1100, U1 MAX3237, U2 ESP-12E, U3 LM1117-3.3

Commit message: Finalised Rev 2 of PCB.
Parts:
- removed the ? at (132.3, 94.5)
- removed the ? at (130.9, 82.8)
- removed the ? at (168.5, 82.3)
- removed the ? at (150.1, 95.1)
- removed the ? at (162.8, 95.2)
- removed the ? at (156.5, 99.2)
- removed the ? at (159.9, 104.1)
- removed the ? at (154.2, 103.5)
- removed the ? at (131.4, 104.9)
- removed the ? at (159.9, 111.4)
- removed the ? at (157.2, 109.0)
- removed the ? at (142.1, 101.5)
- removed the ? at (131.6, 121.3)
- removed the ? at (160.0, 117.9)
- removed the ? at (157.5, 120.0)
- removed the ? at (149.6, 114.6)
- removed the ? at (144.7, 116.6)
- removed the ? at (153.7, 125.2)
- removed the ? at (143.6, 109.0)
- removed the ? at (150.6, 110.5)
- removed the ? at (149.1, 112.8)
- removed the ? at (151.6, 86.4)
- removed the ? at (151.0, 105.9)
- removed the ? at (158.0, 86.4)
- removed the ? at (156.7, 125.7)
- removed the ? at (160.3, 128.0)
- removed the ? at (140.7, 120.4)
- removed the ? at (147.1, 84.6)
- removed the ? at (147.6, 126.4)
- removed the ? at (141.9, 105.3)
- removed the ? at (152.3, 112.1)
- removed the ? at (131.2, 112.8)
- removed the ? at (169.3, 129.3)
- removed the ? at (169.2, 114.7)
- added ?: VIA-0.6mm, Fiducials:VIA-0.6mm, F.Cu at (162.6, 94.7)
- added ?: VIA-0.6mm, Fiducials:VIA-0.6mm, F.Cu at (150.4, 94.0)
- added ?: VIA-0.6mm, Fiducials:VIA-0.6mm, F.Cu at (156.5, 99.6)
- added ?: VIA-0.6mm, Fiducials:VIA-0.6mm, F.Cu at (158.0, 88.1)
- added ?: VIA-0.6mm, Fiducials:VIA-0.6mm, F.Cu at (148.3, 125.0)
- added ?: VIA-0.6mm, Fiducials:VIA-0.6mm, F.Cu at (141.7, 121.9)
- added ?: VIA-0.6mm, Fiducials:VIA-0.6mm, F.Cu at (132.3, 103.9)
- added ?: VIA-0.6mm, Fiducials:VIA-0.6mm, F.Cu at (134.4, 100.1)
- added G***: LOGO, Apple2_bus:CCBYSA, B.Cu at (149.6, 108.2)
- added REF***: OSHW-Symbol_6.7x6mm_SilkScreen, Symbols:OSHW-Symbol_6.7x6mm_SilkScreen, F.Cu at (152.4, 101.9)
Routing:
- net +3V3: track 134.6 -> 155.1 mm
- net GPIO15: track 56.6 -> 40.9 mm, vias 5 -> 2
- net GPIO5: track 37.0 -> 50.4 mm
- net GPIO16: track 41.5 -> 45.2 mm, vias 2 -> 1
- net GPIO10: track 35.3 -> 38.8 mm
- net Net-(R1-Pad2): track 18.5 -> 21.0 mm, vias 0 -> 2
- net DCD: track 20.7 -> 23.1 mm
- net GPIO2: track 35.2 -> 37.5 mm
- net RXD0: track 72.1 -> 74.2 mm, vias 7 -> 2
- net RESET: track 63.7 -> 65.8 mm
- net GPIO13: track 50.9 -> 49.3 mm
- net TXD0: track 76.9 -> 78.1 mm, vias 3 -> 4
- net iDTR: track 36.9 -> 36.1 mm
Other:
- board text added: "(c) 2018 Daniel Jameson"
- board text added: "+5V"
- board text added: "DTR"
- board text added: "FreeFi232"
- board text added: "GND"
- board text added: "HW FLOW"
- board text added: "RESET"
- board text added: "RTS"
- board text added: "RX"
- board text added: "Rev 2"
- board text added: "TX"
- board text added: "WiFi Modem"
- board text added: "https://github.com/stardot/esp8266_modem"
