File: kicad/FreeFi232Large/FreeFi232Large.sch (KiCad schematic (older format))
At the start: 24 parts, among them J1 DB25-Female, J2 3V3-SERIAL, J3 HWFLOW, J4 USB_OTG, J5 ALT-POWER, SW1 B3S-1100, U1 MAX3237, U2 ESP-12E, U3 LM1117-3.3

Commit message: Reverted to KiCAD 4.0.7, revised GPIO pins, BOM added.
Parts:
- removed R2: 470R, Resistors_SMD:R_0805, symbol R
Connections:
- net RESET: now also J2.4 (Pin_4)
- net GPIO14: now reaches U2.5 (GPIO14)
- net GPIO14: now also U1.21 (ROUT1)
- net GPIO10: no longer names the net of U2.20 (GPIO10)
- net GPIO10: no longer U1.21 (ROUT1)
Changed lines of the file:
@@
 Sheet 1 1
 Title "FreeFi232 WiFi Modem"
-Date "2018-06-9"
-Rev "2.1"
+Date "2018-07-04"
+Rev "2.2"
 Comp "(c) 2018 Daniel Jameson"
 Comment1 "License: CC-BY-SA 4.0"
@@
 Text GLabel 6550 3200 0    60   Input ~ 0
 iDTR
-Text GLabel 5800 3300 0    60   Input ~ 0
+Text GLabel 6250 3300 0    60   Input ~ 0
 RESET
 $Comp
@@
 	1    0    0    -1
 $EndComp
-$Comp
-L R R2
-U 1 1 5AF7D55B
-P 6100 3300
-F 0 "R2" V 6180 3300 50  0000 C CNN
-F 1 "470R" V 6100 3300 50  0000 C CNN
-F 2 "Resistors_SMD:R_0805" V 6030 3300 50  0001 C CNN
-F 3 "" H 6100 3300 50  0001 C CNN
-	1    6100 3300
-	0    -1   -1   0
-$EndComp
 Text Notes 7000 3350 0    60   ~ 0
 RTS
@@
 	1550 2600 2300 2600
 Wire Wire Line
-	2300 2600 2300 3800
-Wire Wire Line
-	2300 3800 1550 3800
+	2300 3800 2300 2600
+Wire Wire Line
+	1550 3800 2300 3800
 Wire Wire Line
 	1700 3800 1700 3950
@@
 Wire Wire Line
 	9450 1000 9650 1000
-Wire Wire Line
-	5800 3300 5950 3300
 Wire Wire Line
 	6250 3300 6700 3300
@@
 Wire Wire Line
 	5000 2000 5150 2000
-NoConn ~ 5150 1800
+NoConn ~ 6100 2600
 $Comp
 L MAX3237 U1
@@
 Text GLabel 7000 1900 2    60   Input ~ 0
 GPIO2
-Text GLabel 6200 2750 2    60   Input ~ 0
-GPIO10
 Wire Wire Line
 	6950 1600 7000 1600
@@
 Wire Wire Line
 	6950 1900 7000 1900
-Wire Wire Line
-	6100 2600 6100 2750
-Wire Wire Line
-	6100 2750 6200 2750
 Text GLabel 5550 4550 2    60   Input ~ 0
 GPIO2
@@
 Text GLabel 5550 4950 2    60   Input ~ 0
 GPIO5
-Text GLabel 5550 5150 2    60   Input ~ 0
-GPIO10
 Wire Wire Line
 	5300 4550 5550 4550
@@
 Wire Wire Line
 	7000 5050 7000 5150
+Text GLabel 4550 1800 0    60   Input ~ 0
+GPIO14
+Text GLabel 5550 5150 2    60   Input ~ 0
+GPIO14
+Wire Wire Line
+	4550 1800 5150 1800
 $EndSCHEMATC

Commit message: Schematic corrections - pullup added on RX programming port, GPIOs adjusted.
Parts:
- added R2: 10K, Resistors_SMD:R_0805, symbol R
- J4: footprint Connectors:USB_Micro-B -> Connectors_USB:USB_Micro-B_Molex-105017-0001
Connections:
- net +3V3: now also R2.2
- net RXD0: now also R2.1
- net GPIO12: now reaches U2.6 (GPIO12)
- net GPIO12: now also U1.24 (DIN1)
- net GPIO2: no longer names the net of U2.11 (GPIO2)
- net GPIO2: no longer U1.24 (DIN1)
Changed lines of the file:
@@
 Sheet 1 1
 Title "FreeFi232 WiFi Modem"
-Date "2018-07-04"
-Rev "2.2"
+Date "2018-07-06"
+Rev "2.4"
 Comp "(c) 2018 Daniel Jameson"
 Comment1 "License: CC-BY-SA 4.0"
@@
 F 0 "J4" H 8950 3900 50  0000 L CNN
 F 1 "USB_OTG" H 8950 3800 50  0000 L CNN
-F 2 "Connectors:USB_Micro-B" H 9300 3400 50  0001 C CNN
+F 2 "Connectors_USB:USB_Micro-B_Molex-105017-0001" H 9300 3400 50  0001 C CNN
 F 3 "" H 9300 3400 50  0001 C CNN
 	1    9150 3450
@@
 Text GLabel 7700 2000 2    60   Input ~ 0
 GPIO15
-Text GLabel 5000 2000 0    60   Input ~ 0
+Text GLabel 4550 2000 0    60   Input ~ 0
 GPIO13
 Text GLabel 7700 1800 2    60   Input ~ 0
@@
 NoConn ~ 6200 2600
 NoConn ~ 6300 2600
-NoConn ~ 5150 1900
+NoConn ~ 6950 1900
 NoConn ~ 5150 1500
 $Comp
@@
 	9400 1950 9650 1950
 Wire Wire Line
-	9650 1950 9650 1750
+	9650 1750 9650 2150
 Wire Wire Line
 	6550 3000 6700 3000
@@
 	1550 2600 2300 2600
 Wire Wire Line
-	2300 3800 2300 2600
-Wire Wire Line
-	1550 3800 2300 3800
+	2300 2600 2300 3800
+Wire Wire Line
+	2300 3800 1550 3800
 Wire Wire Line
 	1700 3800 1700 3950
@@
 Connection ~ 8400 5400
 Connection ~ 9800 2750
-Wire Wire Line
-	5000 2000 5150 2000
 NoConn ~ 6100 2600
 $Comp
@@
 Text GLabel 7350 1700 2    60   Input ~ 0
 GPIO4
-Text GLabel 7000 1900 2    60   Input ~ 0
-GPIO2
+Text GLabel 5000 1900 0    60   Input ~ 0
+GPIO12
 Wire Wire Line
 	6950 1600 7000 1600
 Wire Wire Line
 	6950 1700 7350 1700
-Wire Wire Line
-	6950 1900 7000 1900
 Text GLabel 5550 4550 2    60   Input ~ 0
-GPIO2
+GPIO12
 Text GLabel 5550 4750 2    60   Input ~ 0
 GPIO4
@@
 Wire Wire Line
 	4550 1800 5150 1800
+Wire Wire Line
+	4550 2000 5150 2000
+Wire Wire Line
+	5000 1900 5150 1900
+Text GLabel 8950 2150 0    60   Input ~ 0
+RXD0
+$Comp
+L R R2
+U 1 1 5B3FC61E
+P 9250 2150
+F 0 "R2" V 9330 2150 50  0000 C CNN
+F 1 "10K" V 9250 2150 50  0000 C CNN
+F 2 "Resistors_SMD:R_0805" V 9180 2150 50  0001 C CNN
+F 3 "" H 9250 2150 50  0001 C CNN
+	1    9250 2150
+	0    -1   -1   0
+$EndComp
+Wire Wire Line
+	8950 2150 9100 2150
+Wire Wire Line
+	9650 2150 9400 2150
+Connection ~ 9650 1950
 $EndSCHEMATC

Commit message: Error corrected in schematic and PCB. Gerbers updated.
Connections:
- net +3V3: no longer R2.2
- net GND: now also R2.2
Changed lines of the file:
@@
 	9400 1750 9650 1750
-Wire Wire Line
-	9400 1950 9650 1950
-Wire Wire Line
-	9650 1750 9650 2150
 Wire Wire Line
 	6550 3000 6700 3000
@@
 	1550 2600 2300 2600
 Wire Wire Line
-	2300 2600 2300 3800
-Wire Wire Line
-	2300 3800 1550 3800
+	2300 3800 2300 2600
+Wire Wire Line
+	1550 3800 2300 3800
 Wire Wire Line
 	1700 3800 1700 3950
@@
 Wire Wire Line
 	9650 2150 9400 2150
-Connection ~ 9650 1950
+Wire Wire Line
+	9400 1950 9650 1950
+Wire Wire Line
+	9650 1950 9650 1750
+$Comp
+L GND #PWR?
+U 1 1 5B3FDC45
+P 9650 2150
+F 0 "#PWR?" H 9650 1900 50  0001 C CNN
+F 1 "GND" H 9650 2000 50  0000 C CNN
+F 2 "" H 9650 2150 50  0001 C CNN
+F 3 "" H 9650 2150 50  0001 C CNN
+	1    9650 2150
+	1    0    0    -1
+$EndComp
 $EndSCHEMATC

Commit message: Version 2.5 of PCB/Schematic - current limiting resistor between MAX3237 and ESP12
Parts:
- R2: value 10K -> 470R
Connections:
- net GND: no longer R2.2
- net RXD0: no longer U1.18 (ROUT3)
- new net RXD0A: R2.2, U1.18 (ROUT3)
Changed lines of the file:
@@
 Sheet 1 1
 Title "FreeFi232 WiFi Modem"
-Date "2018-07-06"
-Rev "2.4"
+Date "2018-07-25"
+Rev "2.5"
 Comp "(c) 2018 Daniel Jameson"
 Comment1 "License: CC-BY-SA 4.0"
@@
 Tx
 Text GLabel 5550 5750 2    60   Input ~ 0
-RXD0
+RXD0A
 Text GLabel 3450 5950 0    60   Input ~ 0
 Rx
@@
 P 9250 2150
 F 0 "R2" V 9330 2150 50  0000 C CNN
-F 1 "10K" V 9250 2150 50  0000 C CNN
+F 1 "470R" V 9250 2150 50  0000 C CNN
 F 2 "Resistors_SMD:R_0805" V 9180 2150 50  0001 C CNN
 F 3 "" H 9250 2150 50  0001 C CNN
@@
 Wire Wire Line
 	9650 1950 9650 1750
-$Comp
-L GND #PWR?
-U 1 1 5B3FDC45
-P 9650 2150
-F 0 "#PWR?" H 9650 1900 50  0001 C CNN
-F 1 "GND" H 9650 2000 50  0000 C CNN
-F 2 "" H 9650 2150 50  0001 C CNN
-F 3 "" H 9650 2150 50  0001 C CNN
-	1    9650 2150
-	1    0    0    -1
-$EndComp
+Text GLabel 9650 2150 2    60   Input ~ 0
+RXD0A
 $EndSCHEMATC
